Commit message: rename /iiwa_bringup to /lbr_bringup

File: lbr_bringup/urdf/iiwa14.urdf (robot description, URDF)
Before this commit: robot iiwa14, 9 links, 8 joints
Links:
- link base_iiwa: geometry collision mesh filename=package://lbr_bringup/meshes/iiwa14/collision/link_0.stl; visual mesh filename=package://lbr_bringup/meshes/iiwa14/visual/link_0.stl
- link link_1: geometry collision mesh filename=package://lbr_bringup/meshes/iiwa14/collision/link_1.stl; visual mesh filename=package://lbr_bringup/meshes/iiwa14/visual/link_1.stl
- link link_2: geometry collision mesh filename=package://lbr_bringup/meshes/iiwa14/collision/link_2.stl; visual mesh filename=package://lbr_bringup/meshes/iiwa14/visual/link_2.stl
- link link_3: geometry collision mesh filename=package://lbr_bringup/meshes/iiwa14/collision/link_3.stl; visual mesh filename=package://lbr_bringup/meshes/iiwa14/visual/link_3.stl
- link link_4: geometry collision mesh filename=package://lbr_bringup/meshes/iiwa14/collision/link_4.stl; visual mesh filename=package://lbr_bringup/meshes/iiwa14/visual/link_4.stl
- link link_5: geometry collision mesh filename=package://lbr_bringup/meshes/iiwa14/collision/link_5.stl; visual mesh filename=package://lbr_bringup/meshes/iiwa14/visual/link_5.stl
- link link_6: geometry collision mesh filename=package://lbr_bringup/meshes/iiwa14/collision/link_6.stl; visual mesh filename=package://lbr_bringup/meshes/iiwa14/visual/link_6.stl
- link link_7: geometry collision mesh filename=package://lbr_bringup/meshes/iiwa14/collision/link_7.stl; visual mesh filename=package://lbr_bringup/meshes/iiwa14/visual/link_7.stl

File: lbr_bringup/urdf/iiwa7.urdf (robot description, URDF)
Before this commit: robot iiwa7, 9 links, 8 joints
Links:
- link base_iiwa: geometry collision mesh filename=package://lbr_bringup/meshes/iiwa7/collision/link_0.stl; visual mesh filename=package://lbr_bringup/meshes/iiwa7/visual/link_0.dae
- link link_1: geometry collision mesh filename=package://lbr_bringup/meshes/iiwa7/collision/link_1.stl; visual mesh filename=package://lbr_bringup/meshes/iiwa7/visual/link_1.dae
- link link_2: geometry collision mesh filename=package://lbr_bringup/meshes/iiwa7/collision/link_2.stl; visual mesh filename=package://lbr_bringup/meshes/iiwa7/visual/link_2.dae
- link link_3: geometry collision mesh filename=package://lbr_bringup/meshes/iiwa7/collision/link_3.stl; visual mesh filename=package://lbr_bringup/meshes/iiwa7/visual/link_3.dae
- link link_4: geometry collision mesh filename=package://lbr_bringup/meshes/iiwa7/collision/link_4.stl; visual mesh filename=package://lbr_bringup/meshes/iiwa7/visual/link_4_y_z.obj
- link link_5: geometry collision mesh filename=package://lbr_bringup/meshes/iiwa7/collision/link_5.stl; visual mesh filename=package://lbr_bringup/meshes/iiwa7/visual/link_5.dae
- link link_6: geometry collision mesh filename=package://lbr_bringup/meshes/iiwa7/collision/link_6.stl; visual mesh filename=package://lbr_bringup/meshes/iiwa7/visual/link_6.dae
- link link_7: geometry collision mesh filename=package://lbr_bringup/meshes/iiwa7/collision/link_7.stl; visual mesh filename=package://lbr_bringup/meshes/iiwa7/visual/link_7.dae
