Commit message: Fix view robot URDF model in Rviz2

File: lbr_description/urdf/iiwa14.urdf (robot description, URDF)
Before this commit: robot iiwa14, 9 links, 8 joints
Links:
- link base_iiwa: geometry collision mesh filename=package://lbr_description/meshes/iiwa14_white/collision/lin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; visual mesh filename=package://lbr_description/meshes/iiwa14_white/visual/link_0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
- link link_1: geometry collision mesh filename=package://lbr_description/meshes/iiwa14_white/collision/lin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; visual mesh filename=package://lbr_description/meshes/iiwa14_white/visual/link_1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
- link link_2: geometry collision mesh filename=package://lbr_description/meshes/iiwa14_white/collision/lin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; visual mesh filename=package://lbr_description/meshes/iiwa14_white/visual/link_2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
- link link_3: geometry collision mesh filename=package://lbr_description/meshes/iiwa14_white/collision/lin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; visual mesh filename=package://lbr_description/meshes/iiwa14_white/visual/link_3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
- link link_4: geometry collision mesh filename=package://lbr_description/meshes/iiwa14_white/collision/lin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; visual mesh filename=package://lbr_description/meshes/iiwa14_white/visual/link_4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
- link link_5: geometry collision mesh filename=package://lbr_description/meshes/iiwa14_white/collision/lin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; visual mesh filename=package://lbr_description/meshes/iiwa14_white/visual/link_5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
- link link_6: geometry collision mesh filename=package://lbr_description/meshes/iiwa14_white/collision/lin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; visual mesh filename=package://lbr_description/meshes/iiwa14_white/visual/link_6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
- link link_7: geometry collision mesh filename=package://lbr_description/meshes/iiwa14_white/collision/lin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; visual mesh filename=package://lbr_description/meshes/iiwa14_white/visual/link_7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

File: lbr_description/urdf/iiwa7.urdf (robot description, URDF)
Before this commit: robot iiwa7, 9 links, 8 joints
Links:
- link base_iiwa: geometry collision mesh filename=package://lbr_description/meshes/iiwa7_white/collision/link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; visual mesh filename=package://lbr_description/meshes/iiwa7_white/visual/link_0.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
- link link_1: geometry collision mesh filename=package://lbr_description/meshes/iiwa7_white/collision/link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; visual mesh filename=package://lbr_description/meshes/iiwa7_white/visual/link_1.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
- link link_2: geometry collision mesh filename=package://lbr_description/meshes/iiwa7_white/collision/link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; visual mesh filename=package://lbr_description/meshes/iiwa7_white/visual/link_2.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
- link link_3: geometry collision mesh filename=package://lbr_description/meshes/iiwa7_white/collision/link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; visual mesh filename=package://lbr_description/meshes/iiwa7_white/visual/link_3.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
- link link_4: geometry collision mesh filename=package://lbr_description/meshes/iiwa7_white/collision/link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; visual mesh filename=package://lbr_description/meshes/iiwa7_white/visual/link_4_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
- link link_5: geometry collision mesh filename=package://lbr_description/meshes/iiwa7_white/collision/link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; visual mesh filename=package://lbr_description/meshes/iiwa7_white/visual/link_5.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
- link link_6: geometry collision mesh filename=package://lbr_description/meshes/iiwa7_white/collision/link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; visual mesh filename=package://lbr_description/meshes/iiwa7_white/visual/link_6.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
- link link_7: geometry collision mesh filename=package://lbr_description/meshes/iiwa7_white/collision/link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; visual mesh filename=package://lbr_description/meshes/iiwa7_white/visual/link_7.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
